File: boards/controller-board/untitled.kicad_sch (KiCad schematic)
At the start: 144 parts, among them IC10 A6214KLKTR-T, IC11 A6214KLKTR-T, IC12 A6214KLKTR-T, IC13 A6214KLKTR-T, IC14 A6214KLKTR-T, IC3 A6214KLKTR-T, IC4 A6214KLKTR-T, IC5 A6214KLKTR-T, IC6 A6214KLKTR-T, IC7 A6214KLKTR-T, IC8 A6214KLKTR-T, IC9 A6214KLKTR-T

Commit message: cleaned up controller schematic
Parts:
- renumbered C25 to C38, C70 to C39, C74 to C40, C66 to C43, C26 to C44, C71 to C45, C75 to C46, C52 to C47, C53 to C48, C67 to C49, C34 to C50, C72 to C51, C76 to C52, C78 to C53, C79 to C54, C68 to C55, C36 to C56, C73 to C57, C77 to C58, C80 to C59, C81 to C60, C69 to C61, C49 to C62, C82 to C63, C56 to C64, C61 to C65, C90 to C66, C95 to C67, C50 to C68, C83 to C69, C88 to C70, C86 to C71, C91 to C72, C97 to C73, C54 to C74, C84 to C75, C92 to C76, C87 to C77, C93 to C78, C98 to C79, C55 to C80, C85 to C81, C96 to C82, C89 to C83, C94 to C84, C99 to C85, D5 to D41, D93 to D42, D97 to D43, D34 to D44, D38 to D45, D89 to D46, D6 to D47, D7 to D48, D94 to D49, D95 to D50, D98 to D51, D99 to D52, D57 to D53, D58 to D54, D59 to D55, D60 to D56, D90 to D57, D91 to D58, D8 to D59, D96 to D60, D100 to D61, D65 to D62, D66 to D63, D92 to D64, D39 to D65, D63 to D66, D69 to D67, D74 to D68, D104 to D69, D108 to D70, D41 to D71, D61 to D72, D64 to D73, D67 to D74, D101 to D75, D102 to D76, D75 to D77, D84 to D78, D105 to D79, D106 to D80, D110 to D81, D111 to D82, D62 to D83, D68 to D84, D109 to D85, D103 to D86, D107 to D87, D112 to D88, IC11 to IC10, IC12 to IC11, IC13 to IC12, IC14 to IC13, IC3 to IC2, IC5 to IC3, IC6 to IC4, IC7 to IC5, IC8 to IC6, IC4 to IC7, IC9 to IC8, IC10 to IC9, L6 to L12, L25 to L13, L26 to L14, L9 to L15, L24 to L17, L17 to L18, L18 to L19, L19 to L20, L27 to L21, L28 to L22, L29 to L23, R14 to R23, R39 to R24, R41 to R25, R28 to R26, R29 to R27, R37 to R28, R18 to R29, R40 to R30, R42 to R31, R43 to R32, R44 to R33, R38 to R34, R30 to R35, R45 to R36, R32 to R37, R47 to R38, R49 to R39, R52 to R40, R31 to R41, R46 to R42, R50 to R43, R48 to R44, R51 to R45, R53 to R46
Other:
- moved on the sheet: C39, C40, C41, C42, C43, C45, C46, C47, C48, C49, C51, C52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

Commit message: redesigned pcb
Parts:
- removed C65, C66, C67: 33u TBD, symbol Device:C_Small
- removed C68, C69, C70, C71, C72, C73: 1u, symbol Device:C_Small
- removed C74, C75, C76, C77, C78, C79: 100n TBD, symbol Device:C_Small
- removed C80, C81, C82, C83, C84, C85: 100n, symbol Device:C_Small
- removed D42, D43, D44, D45, D46, D65, D66, D67, D68, D69, D70: NSR0320, symbol Device:D_Schottky
- removed L13, L14, L15, L16, L17, L19, L20, L21, L22, L23: 22u, symbol Device:L_Small
- added C11, C12, C13, C14, C20, C21, C22, C23, C24, C25, C26, C27, C28, C29, C30, C31, C33, C34, C35, C36, C37: 100n, oresat-passives:0402-C, symbol Device:C_Small
- added C32: 470u, Capacitor_SMD:CP_Elec_10x12.5, symbol Device:C_Small
- added D1, D10, D11, D2, D3, D4, D5, D6, D7, D8, D9: VS-10MQ060NTRPBF, Diode_SMD:D_SMA, symbol Device:D_Schottky
- added L10, L11, L2, L3, L4, L5, L6, L7, L8, L9: 47u, Inductor_SMD:L_Coilcraft_MSS1048-XXX, symbol Device:L_Small
- added R11, R14, R15, R16, R17, R18, R19, R20, R21, R22, R6: .560, oresat-passives:0402-C, symbol Device:R_Small_US
- added R47: 1k, oresat-passives:0603-C, symbol Device:R_Small_US
- C38, C39, C40: value 33u TBD -> 100n; footprint (none) -> oresat-passives:0402-C
- C41, C42, C43, C62, C64: value 33u TBD -> 10u; footprint (none) -> oresat-passives:1206-C
- C44, C45, C46, C47, C48, C49, R23, R24, R25, R26, R27, R28, R35: footprint (none) -> oresat-passives:0603-C
- C50, C51: value 100n TBD -> 10u; footprint (none) -> oresat-passives:1206-C
- C52, C53, C54, C55: value 100n TBD -> 1u; footprint (none) -> oresat-passives:0603-C
- C56: value 100n -> 1u; footprint (none) -> oresat-passives:0603-C
- C57, C58, C59, C60, C61: value 100n -> 10u; footprint (none) -> oresat-passives:1206-C
- C63: value 33u TBD -> 1u; footprint (none) -> oresat-passives:0603-C
- D41: value NSR0320 -> VS-10MQ060NTRPBF; footprint (none) -> Diode_SMD:D_SMA
- L12, L18: value 22u -> 47u; footprint (none) -> Inductor_SMD:L_Coilcraft_MSS1048-XXX
- R29, R30, R31, R32, R34: value .576 -> 95.3k; footprint (none) -> oresat-passives:0603-C
- R33: value .576 -> .560; footprint (none) -> oresat-passives:0402-C
- R36, R37, R38, R39, R40: value 95.3k -> 1k; footprint (none) -> oresat-passives:0603-C
- R41, R42, R43, R44, R45, R46: value .576 -> 1k; footprint (none) -> oresat-passives:0603-C
Connections:
- net GND: now also C50.2, C51.2, C52.2, C53.2, C54.2, C55.2, C22.2, C26.2, C28.2, C30.2, C31.2, C32.2, C33.2, C34.2, C35.2, C37.2, D1.2 (A), D10.2 (A), D11.2 (A), D2.2 (A), D3.2 (A), D4.2 (A), D5.2 (A), D6.2 (A), D7.2 (A), D8.2 (A), D9.2 (A)
- net VCC: now also C50.1, C51.1, C57.1, C58.1, C59.1, C60.1, C61.1, R29.1, R30.1, R31.1, R32.1, R34.1, R41.1, R42.1, R43.1, R44.1, R45.1, R46.1, C32.1, R47.1; no longer C38.1, C39.1, C40.1, C63.1
- net at IC11.10 (SW): now also C25.1, D9.1 (K), L11.1
- net at IC11.8 (CSH): now also L11.2, R21.1; no longer R44.1
- net at C52.1: now also IC9.5 (VCC); no longer IC4.10 (SW)
- net at IC10.2 (TON): now also R31.2; no longer R37.2
- net at D75.2 (A), IC10.7 (CSL): now also C40.1, R20.2; no longer R43.2
- net at IC9.8 (CSH): now also L2.2, R18.1; no longer R42.1
- net at D73.2 (A), IC9.7 (CSL): now also C38.1, R18.2; no longer R42.2
- net at D71.2 (A), IC8.7 (CSL): now also C37.1, R19.2; no longer R41.2
- net at IC13.10 (SW): now also C24.1, D11.1 (K), L9.1
- net at IC13.8 (CSH): now also R33.1, L9.2; no longer R46.1
- net at IC12.8 (CSH): now also L10.2, R22.1; no longer R45.1
- net at D79.2 (A), IC12.7 (CSL): now also C30.1, R22.2; no longer R45.2
- net at IC7.10 (SW): now also C11.1, D1.1 (K), L6.1; no longer C55.1
- net at IC7.9 (BOOT): now also C11.2; no longer C55.2
- net at R36.2: now also IC2.3 (EN/PWM); no longer IC9.2 (TON)
- net at IC5.10 (SW): now also C21.1, D6.1 (K), L3.1; no longer C53.1
- net at IC5.9 (BOOT): now also C21.2; no longer C53.2
- net at IC9.10 (SW): now also C20.1, D5.1 (K), L2.1
- net at IC9.9 (BOOT): now also C20.2
- net at IC7.8 (CSH): now also L6.2, R11.1; no longer R34.1
- net at D57.2 (A), IC7.7 (CSL): now also C35.1, R11.2; no longer C61.1, R34.2
- net at D81.2 (A), IC13.7 (CSL): now also R33.2, C31.1; no longer R46.2
- net at D53.2 (A), IC5.7 (CSL): now also C39.1, R17.2; no longer C59.1, R32.2
- net at D51.2 (A), IC4.7 (CSL): now also C33.1, R15.2; no longer C58.1, R31.2
- net at D47.2 (A), IC2.7 (CSL): now also C28.1, R6.2; no longer C56.1, R29.2
- net at IC6.10 (SW): now also C23.1, D7.1 (K), L4.1; no longer C54.1
- net at IC6.5 (VCC): now also C47.1; no longer C48.1
- net at D55.2 (A), IC6.7 (CSL): now also C22.1, R16.2; no longer C60.1, R33.2
- net at IC6.8 (CSH): now also L4.2, R16.1; no longer R33.1
- net at IC6.9 (BOOT): now also C23.2; no longer C54.2
- net at R25.2: now also IC3.2 (TON); no longer IC4.2 (TON)
- net at IC4.8 (CSH): now also L8.2, R15.1; no longer R31.1
- net at IC4.9 (BOOT): now also C13.2; no longer C52.2
- net at R40.2: now also IC8.3 (EN/PWM); no longer IC13.2 (TON)
- net at IC8.10 (SW), L18.1: now also C14.1, D4.1 (K)
- net at IC8.9 (BOOT): now also C14.2
- net at IC12.10 (SW): now also C29.1, D10.1 (K), L10.1
- net at R39.2: now also IC4.3 (EN/PWM); no longer IC12.2 (TON)
- net at IC12.5 (VCC): now also C55.1
- net at IC12.9 (BOOT): now also C29.2
- net at IC5.8 (CSH): now also L3.2, R17.1; no longer R32.1
- net at IC10.5 (VCC): now also C53.1
- net at IC8.8 (CSH), L18.2: now also R19.1; no longer R41.1
- net at D41.1 (K), IC2.10 (SW): now also C36.1, L5.1; no longer C50.1, L12.1
- net at IC2.9 (BOOT): now also C36.2; no longer C50.2
- net at IC3.10 (SW): now also C12.1, D2.1 (K), L7.1; no longer C51.1
- net at IC3.9 (BOOT): now also C12.2; no longer C51.2
- net at D77.2 (A), IC11.7 (CSL): now also C26.1, R21.2; no longer R44.2
- net at R26.2: now also IC4.2 (TON); no longer IC5.2 (TON)
- net at IC10.10 (SW): now also L12.1, C27.1, D8.1 (K)
- net at IC8.2 (TON): now also R30.2; no longer R35.2
- net at IC8.5 (VCC): now also C63.1
- net at IC11.2 (TON): now also R32.2; no longer R38.2
- net at IC11.5 (VCC): now also C54.1
- net at IC11.9 (BOOT): now also C25.2
- net at IC7.5 (VCC): now also C45.1; no longer C49.1
- net at IC13.9 (BOOT): now also C24.2
- net at IC3.5 (VCC): now also C49.1; no longer C45.1
- net at IC7.2 (TON): now also R24.2; no longer R28.2
- net at IC5.5 (VCC): now also C48.1; no longer C47.1
- net at IC10.8 (CSH): now also L12.2, R20.1; no longer R43.1
- net at IC10.9 (BOOT): now also C27.2
- net at D49.2 (A), IC3.7 (CSL): now also C34.1, R14.2; no longer C57.1, R30.2
- net at IC3.8 (CSH): now also L7.2, R14.1; no longer R30.1
- net at IC13.5 (VCC): now also C56.1
- removed net +5V: IC10.3 (EN/PWM), IC11.3 (EN/PWM), IC12.3 (EN/PWM), IC13.3 (EN/PWM), IC2.3 (EN/PWM), IC3.3 (EN/PWM), IC4.3 (EN/PWM), IC5.3 (EN/PWM), IC6.3 (EN/PWM), IC7.3 (EN/PWM), IC8.3 (EN/PWM), IC9.3 (EN/PWM)
- new net: IC9.2 (TON), R29.2
- new net: IC9.3 (EN/PWM), R41.2
- new net: IC2.8 (CSH), L5.2, R6.1
- new net: IC12.3 (EN/PWM), R46.2
- new net: IC6.3 (EN/PWM), R43.2
- new net: C13.1, D3.1 (K), IC4.10 (SW), L8.1
- new net: IC12.2 (TON), R34.2
- new net: IC13.3 (EN/PWM), R47.2
- new net: IC11.3 (EN/PWM), R45.2
- new net: IC10.3 (EN/PWM), R44.2
- new net: IC7.3 (EN/PWM), R37.2
- new net: IC5.2 (TON), R28.2
- new net: IC5.3 (EN/PWM), R42.2
- new net: IC3.3 (EN/PWM), R38.2
- new net: IC13.2 (TON), R35.2
Other:
- note added: "Bypass Capacitor (parallel caps from LED drivers in one)"
- note added: "check buck conv. diode. better alternative (smaller voltage/smaller footprint)?"
- moved on the sheet: C46, D41, D47, D48, D49, D50, D51, D52, D53, D54, D55, D56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

Commit message: changed footprint on sense resistors, adjusted traces
Parts:
- C22, C26, C28, C30, C31, C33, C34, C35, C37, C38, C39, C40: footprint oresat-passives:0402-C -> oresat-passives:0603-C
- R11, R14, R15, R16, R17, R18, R19, R20, R21, R22, R33, R6: value .560 -> .576; footprint oresat-passives:0402-C -> oresat-passives:0603-C
Other:
- note added: "add 100k pull-down resistor for adim pins"
Changed lines of the file:
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@@
 		)
 	)
+	(text "add 100k pull-down resistor for adim pins"
+		(exclude_from_sim no)
+		(at 100.33 40.894 0)
+		(effects
+			(font
+				(size 1.27 1.27)
+			)
+		)
+	)
 	(text "Red LED Channel"
 		(exclude_from_sim no)
@@
 			)
 		)
-		(property "Footprint" "oresat-passives:0402-C"
+		(property "Footprint" "oresat-passives:0603-C"
 			(at 170.18 160.02 0)
 			(effects
@@
 			)
 		)
-		(property "Value" ".560"
+		(property "Value" ".576"
 			(at 163.322 214.6301 0)
 			(effects
@@
 			)
 		)
-		(property "Footprint" "oresat-passives:0402-C"
+		(property "Footprint" "oresat-passives:0603-C"
 			(at 170.18 213.36 0)
 			(effects
@@
 			)
 		)
-		(property "Value" ".560"
+		(property "Value" ".576	"
 			(at 322.072 220.9801 0)
 			(effects
@@
 			)
 		)
-		(property "Footprint" "oresat-passives:0402-C"
+		(property "Footprint" "oresat-passives:0603-C"
 			(at 328.93 219.71 0)
 			(effects
@@
 			)
 		)
-		(property "Value" ".560"
+		(property "Value" ".576"
 			(at 484.632 153.6701 0)
 			(effects
@@
 			)
 		)
-		(property "Footprint" "oresat-passives:0402-C"
+		(property "Footprint" "oresat-passives:0603-C"
 			(at 491.49 152.4 0)
 			(effects
@@
 			)
 		)
-		(property "Value" ".560"
+		(property "Value" ".576"
 			(at 484.632 279.4001 0)
 			(effects
@@
 			)
 		)
-		(property "Footprint" "oresat-passives:0402-C"
+		(property "Footprint" "oresat-passives:0603-C"
 			(at 491.49 278.13 0)
 			(effects
@@
 			)
 		)
-		(property "Footprint" "oresat-passives:0402-C"
+		(property "Footprint" "oresat-passives:0603-C"
 			(at 170.18 223.52 0)
 			(effects
@@
 			)
 		)
-		(property "Footprint" "oresat-passives:0402-C"
+		(property "Footprint" "oresat-passives:0603-C"
 			(at 328.93 96.52 0)
 			(effects
@@
 			)
 		)
-		(property "Footprint" "oresat-passives:0402-C"
+		(property "Footprint" "oresat-passives:0603-C"
 			(at 328.93 292.1 0)
 			(effects
@@
 			)
 		)
-		(property "Footprint" "oresat-passives:0402-C"
+		(property "Footprint" "oresat-passives:0603-C"
 			(at 491.49 288.29 0)
 			(effects
@@
 			)
 		)
-		(property "Footprint" "oresat-passives:0402-C"
+		(property "Footprint" "oresat-passives:0603-C"
 			(at 170.18 95.25 0)
 			(effects
@@
 			)
 		)
-		(property "Value" ".560"
+		(property "Value" ".576"
 			(at 484.632 215.9001 0)
 			(effects
@@
 			)
 		)
-		(property "Footprint" "oresat-passives:0402-C"
+		(property "Footprint" "oresat-passives:0603-C"
 			(at 491.49 214.63 0)
 			(effects
@@
 			)
 		)
-		(property "Value" ".560"
+		(property "Value" ".576"
 			(at 322.072 156.2101 0)
 			(effects
@@
 			)
 		)
-		(property "Footprint" "oresat-passives:0402-C"
+		(property "Footprint" "oresat-passives:0603-C"
 			(at 328.93 154.94 0)
 			(effects
@@
 			)
 		)
-		(property "Value" ".560"
+		(property "Value" ".576"
 			(at 163.322 151.1301 0)
 			(effects
@@
 			)
 		)
-		(property "Footprint" "oresat-passives:0402-C"
+		(property "Footprint" "oresat-passives:0603-C"
 			(at 170.18 149.86 0)
 			(effects
@@
 			)
 		)
-		(property "Footprint" "oresat-passives:0402-C"
+		(property "Footprint" "oresat-passives:0603-C"
 			(at 491.49 162.56 0)
 			(effects
@@
 			)
 		)
-		(property "Footprint" "oresat-passives:0402-C"
+		(property "Footprint" "oresat-passives:0603-C"
 			(at 170.18 285.75 0)
 			(effects
@@
 			)
 		)
-		(property "Value" ".560"
+		(property "Value" ".576	"
 			(at 163.322 86.3601 0)
 			(effects
@@
 			)
 		)
-		(property "Footprint" "oresat-passives:0402-C"
+		(property "Footprint" "oresat-passives:0603-C"
 			(at 170.18 85.09 0)
 			(effects
@@
 			)
 		)
-		(property "Footprint" "oresat-passives:0402-C"
+		(property "Footprint" "oresat-passives:0603-C"
 			(at 491.49 224.79 0)
 			(effects
@@
 			)
 		)
-		(property "Footprint" "oresat-passives:0402-C"
+		(property "Footprint" "oresat-passives:0603-C"
 			(at 491.49 97.79 0)
 			(effects
@@
 			)
 		)
-		(property "Footprint" "oresat-passives:0402-C"
+		(property "Footprint" "oresat-passives:0603-C"
 			(at 328.93 165.1 0)
 			(effects
@@
 			)
 		)
-		(property "Value" ".560"
+		(property "Value" ".576"
 			(at 484.632 88.9001 0)
 			(effects
@@
 			)
 		)
-		(property "Footprint" "oresat-passives:0402-C"
+		(property "Footprint" "oresat-passives:0603-C"
 			(at 491.49 87.63 0)
 			(effects
@@
 			)
 		)
-		(property "Value" ".560"
+		(property "Value" ".576"
 			(at 322.072 283.2101 0)
 			(effects
@@
 			)
 		)
-		(property "Footprint" "oresat-passives:0402-C"
+		(property "Footprint" "oresat-passives:0603-C"
 			(at 328.93 281.94 0)
 			(effects
@@
 			)
 		)
-		(property "Value" ".560"
+		(property "Value" ".576"
 			(at 322.072 87.6301 0)
 			(effects
@@
 			)
 		)
-		(property "Footprint" "oresat-passives:0402-C"
+		(property "Footprint" "oresat-passives:0603-C"
 			(at 328.93 86.36 0)
 			(effects
@@
 			)
 		)
-		(property "Value" ".560"
+		(property "Value" ".576"
 			(at 163.322 276.8601 0)
 			(effects
@@
 			)
 		)
-		(property "Footprint" "oresat-passives:0402-C"
+		(property "Footprint" "oresat-passives:0603-C"
 			(at 170.18 275.59 0)
 			(effects
@@
 			)
 		)
-		(property "Footprint" "oresat-passives:0402-C"
+		(property "Footprint" "oresat-passives:0603-C"
 			(at 328.93 229.87 0)
 			(effects
