File: boards/controller-board/controller-board.kicad_pcb (KiCad board)
At the start: 2 copper layers, 130 x 115 mm, 213 parts, among them IC10 A6214KLKTR-T, IC11 A6214KLKTR-T, IC12 A6214KLKTR-T, IC13 A6214KLKTR-T, IC2 A6214KLKTR-T, IC3 A6214KLKTR-T, IC4 A6214KLKTR-T, IC5 A6214KLKTR-T, IC6 A6214KLKTR-T, IC7 A6214KLKTR-T, IC8 A6214KLKTR-T, IC9 A6214KLKTR-T, J1 Conn_01x02, J2 Conn_01x02, J3 Conn_01x02, J4 Conn_01x02, J5 Conn_01x03, J6 Conn_01x02, Q1 PMV45EN, Q2 Goford_G11S_20V_11A, SW1 EG1271, U1 LTC3624, U2 ADS1015IRUGR, U3 ADS1015IRUGR, U4 RPi_Pico, U5 MCP4728

Commit message: minor changes to tracks and zones
Parts:
- moved L1 0.29 mm to (154.7, 54.1)
- moved C8 0.25 mm to (153.9, 48.9)
- moved C63 0.06 mm to (100.1, 143.0)
- moved C10 0.05 mm to (158.9, 52.0)
Routing:
- net GND: track 0.37 -> 1.25 mm, vias 322 -> 326
- net Net-(U1-INTVcc): track 8.99 -> 8.24 mm
Changed lines of the file:
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@@
 	(footprint "Capacitor_SMD:C_1210_3225Metric"
 		(layer "F.Cu")
-		(at 157.17 48.88 90)
+		(at 157.15 48.92 90)
 		(descr "Capacitor SMD 1210 (3225 Metric), square (rectangular) end terminal, IPC_7351 nominal, (Body size source: IPC-SM-782 page 76, https://www.pcb-3d.com/wordpress/wp-content/uploads/ipc-sm-782a_amendment_1_and_2.pdf), generated with kicad-footprint-generator")
 		(tags "capacitor")
@@
 	(footprint "Capacitor_SMD:C_1210_3225Metric"
 		(layer "F.Cu")
-		(at 153.91 49.15 90)
+		(at 153.9 48.9 90)
 		(descr "Capacitor SMD 1210 (3225 Metric), square (rectangular) end terminal, IPC_7351 nominal, (Body size source: IPC-SM-782 page 76, https://www.pcb-3d.com/wordpress/wp-content/uploads/ipc-sm-782a_amendment_1_and_2.pdf), generated with kicad-footprint-generator")
 		(tags "capacitor")
@@
 	(footprint "oresat-passives:L_ECS-MPI4040"
 		(layer "F.Cu")
-		(at 154.67 54.38 90)
+		(at 154.72 54.09 90)
 		(descr "Inductor SMD 2010 (5025 Metric), square (rectangular) end terminal, IPC_7351 nominal")
 		(tags "inductor")
@@
 	(footprint "Capacitor_SMD:C_0603_1608Metric"
 		(layer "F.Cu")
-		(at 158.86 51.99)
+		(at 158.91 51.98)
 		(descr "Capacitor SMD 0603 (1608 Metric), square (rectangular) end terminal, IPC_7351 nominal, (Body size source: IPC-SM-782 page 76, https://www.pcb-3d.com/wordpress/wp-content/uploads/ipc-sm-782a_amendment_1_and_2.pdf), generated with kicad-footprint-generator")
 		(tags "capacitor")
@@
 	(footprint "oresat-passives:0603-C"
 		(layer "F.Cu")
-		(at 100.02 142.98 180)
+		(at 100.08 143 180)
 		(descr "<b>0603 (metric 1608) tight 'IPC-C'</b>\n<br>In house package for minimum spacing based on IPC-7351B.")
 		(property "Reference" "C63"
@@
 	)
 	(segment
+		(start 167.32 55.55)
+		(end 168.745 55.55)
+		(width 2)
+		(layer "F.Cu")
+		(net 1)
+	)
+	(segment
 		(start 186.58 115.42)
 		(end 185.26 116.74)
@@
 	)
 	(segment
-		(start 168.585 55.55)
-		(end 170.11 57.075)
-		(width 1)
-		(layer "F.Cu")
-		(net 1)
-	)
-	(segment
 		(start 163.27 56.71)
 		(end 163.27 55.53)
@@
 	)
 	(segment
-		(start 166.96 55.55)
-		(end 168.585 55.55)
-		(width 1)
-		(layer "F.Cu")
-		(net 1)
-	)
-	(segment
 		(start 93.3 115.34)
 		(end 102.64 115.34)
@@
 	)
 	(segment
+		(start 168.745 55.55)
+		(end 170.24 57.045)
+		(width 2)
+		(layer "F.Cu")
+		(net 1)
+	)
+	(segment
 		(start 197.365397 115.42)
 		(end 186.58 115.42)
@@
 		(net 2)
 	)
+	(segment
+		(start 158.1 55.27)
+		(end 158.98 55.27)
+		(width 0.25)
+		(layer "F.Cu")
+		(net 2)
+	)
 	(via
 		(at 185 92)
@@
 	)
 	(via
+		(at 188.73 75.05)
+		(size 0.508)
+		(drill 0.254)
+		(layers "F.Cu" "B.Cu")
+		(free yes)
+		(net 2)
+	)
+	(via
 		(at 176 112)
 		(size 0.508)
@@
 	)
 	(via
+		(at 190.5 75.82)
+		(size 0.508)
+		(drill 0.254)
+		(layers "F.Cu" "B.Cu")
+		(free yes)
+		(net 2)
+	)
+	(via
 		(at 197.74 105.09)
 		(size 0.508)
@@
 	)
 	(via
+		(at 189.87 75.02)
+		(size 0.508)
+		(drill 0.254)
+		(layers "F.Cu" "B.Cu")
+		(free yes)
+		(net 2)
+	)
+	(via
 		(at 192.786 97.282)
 		(size 0.508)
@@
 	)
 	(via
+		(at 188.73 75.77)
+		(size 0.508)
+		(drill 0.254)
+		(layers "F.Cu" "B.Cu")
+		(free yes)
+		(net 2)
+	)
+	(via
 		(at 99.97 112.21)
 		(size 0.508)
@@
 	)
 	(segment
-		(start 158.1 54.27)
-		(end 151.39 54.27)
+		(start 151.8428 54.13)
+		(end 151.2228 53.51)
 		(width 0.25)
 		(layer "F.Cu")
@@
 	)
 	(segment
-		(start 151.39 54.27)
-		(end 151.2228 54.1028)
+		(start 157.692576 54.27)
+		(end 157.552576 54.13)
 		(width 0.25)
 		(layer "F.Cu")
@@
 	)
 	(segment
-		(start 151.2228 54.1028)
-		(end 151.2228 53.51)
+		(start 151.2228 52.065)
+		(end 151.2178 52.06)
 		(width 0.25)
 		(layer "F.Cu")
@@
 	)
 	(segment
-		(start 151.2228 52.065)
-		(end 151.2178 52.06)
+		(start 157.552576 54.13)
+		(end 151.8428 54.13)
 		(width 0.25)
 		(layer "F.Cu")
@@
 	)
 	(segment
+		(start 157.623496 54.77)
+		(end 157.385896 54.5324)
+		(width 0.25)
+		(layer "F.Cu")
+		(net 118)
+	)
+	(segment
 		(start 158.1 54.77)
-		(end 152.27 54.77)
+		(end 157.623496 54.77)
 		(width 0.25)
 		(layer "F.Cu")
@@
 	)
 	(segment
-		(start 151.88 55.16)
+		(start 151.8504 54.5324)
 		(end 151.2228 55.16)
 		(width 0.25)
@@
 	)
 	(segment
-		(start 152.27 54.77)
-		(end 151.88 55.16)
+		(start 157.385896 54.5324)
+		(end 151.8504 54.5324)
 		(width 0.25)
 		(layer "F.Cu")
@@
 		(polygon
 			(pts
-				(xy 109.194991 152.905529) (xy 109.194991 150.496532) (xy 107.130194 150.496532) (xy 107.130194 152.905529)
+				(xy 109.194991 152.905529) (xy 109.194991 150.496532) (xy 107.378248 150.496532) (xy 107.378248 152.905529)
 			)
 		)
@@
 		(polygon
 			(pts
-				(xy 160.49 55.025) (xy 161.72 55.025) (xy 161.72 56.413756) (xy 167.75 56.413756) (xy 167.75 54.525)
-				(xy 160.49 54.525)
+				(xy 160.49 55.025) (xy 161.72 55.025) (xy 161.72 56.483756) (xy 167.75 56.483756) (xy 167.75 54.515)
+				(xy 160.49 54.515)
 			)
 		)
