File: boards/controller-board/controller-board-pico.kicad_sch (KiCad schematic)
At the start: 52 parts, among them J2 Conn_01x02, J3 Conn_01x02, J4 Conn_01x02, J5 0470531000, J6 1935161, Q1 PMV45EN, Q2 G11S_20V_11A, U1 XIAO-RP2040-SMD, U2 ADS1015IRUGR, U3 MIC44F19YMME, U5 MCP4728

Commit message: Add halogen driver design variants
Other:
- note added: "Backup N channel for the P channel MOSFET driver circuit"
- note removed: "Backup P ch MOSFET driver circuit"
Changed lines of the file:
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@@
 		)
 	)
-	(text "Backup P ch MOSFET\ndriver circuit"
+	(text "Backup N channel for the \nP channel MOSFET driver circuit"
 		(exclude_from_sim no)
-		(at 244.856 44.958 0)
+		(at 239.522 43.18 0)
 		(effects
 			(font
@@
 					(reference "Q1")
 					(unit 1)
+					(variant
+						(name "Halogen N Channel MOSFET Driver")
+						(dnp no)
+					)
 				)
 			)
@@
 					(reference "R12")
 					(unit 1)
+					(variant
+						(name "Halogen N Channel MOSFET Driver")
+						(dnp no)
+					)
 				)
 			)
@@
 					(reference "C37")
 					(unit 1)
+					(variant
+						(name "Halogen N Channel MOSFET Driver")
+						(dnp yes)
+					)
 				)
 			)
@@
 					(reference "C17")
 					(unit 1)
+					(variant
+						(name "Halogen N Channel MOSFET Driver")
+						(dnp no)
+					)
 				)
 			)
@@
 					(reference "TP24")
 					(unit 1)
+					(variant
+						(name "Halogen N Channel MOSFET Driver")
+						(dnp yes)
+					)
 				)
 			)
@@
 					(reference "U3")
 					(unit 1)
+					(variant
+						(name "Halogen N Channel MOSFET Driver")
+						(dnp yes)
+					)
 				)
 			)
@@
 					(reference "R9")
 					(unit 1)
+					(variant
+						(name "Halogen N Channel MOSFET Driver")
+						(dnp no)
+					)
 				)
 			)
@@
 					(reference "#PWR028")
 					(unit 1)
+					(variant
+						(name "Halogen N Channel MOSFET Driver")
+						(dnp yes)
+					)
 				)
 			)
@@
 					(reference "R13")
 					(unit 1)
+					(variant
+						(name "Halogen N Channel MOSFET Driver")
+						(dnp no)
+					)
 				)
 			)
